Commit message: added launch controll

File: bot_discription/urdf/bumperbot.urdf.xacro (robot description, xacro)
@@ -4,5 +4,5 @@
   <xacro:arg name="is_ignition" default="true"/>
   <!-- Load Simulated or Real Hardware Interfaces -->
-  <!-- <xacro:arg name="is_sim" default="true"/> -->
+  <xacro:arg name="is_sim" default="true"/>
   <!-- Include Gazebo Parameters -->
   <xacro:include filename="$(find bot_discription)/urdf/bumperbot_gazebo.xacro" />
@@ -175,16 +175,3 @@
     <axis xyz="0 0 0" />
   </joint>
-  <!-- <link name="can_link">
-    <visual>
-      <origin xyz="-0.0307 0.0307 0" rpy="1.57 0 0" />
-      <geometry>
-        <mesh filename="package://bot_discription/meshes/can.STL" />
-      </geometry>
-    </visual>
-  </link>
-  <joint name="can_joint" type="fixed">
-    <origin xyz="0 0 0.078" rpy="0 0 0" />
-    <parent link="base_link" />
-    <child link="can_link" />
-  </joint>   -->
 </robot>

File: bot_discription/urdf/bumperbot_gazebo.xacro (robot description, xacro)
@@ -1,4 +1,4 @@
 <?xml version="1.0"?>
-<robot name="bot" xmlns:xacro="http://ros.org/wiki/xacro">
+<robot name="bumperbot" xmlns:xacro="http://ros.org/wiki/xacro">
   <!-- Wheels -->
   <gazebo reference="wheel_left_link">
@@ -47,9 +47,8 @@
       </plugin>
     </xacro:if>
-  </gazebo>
     <!-- ROS 2 Iron or above -->
     <xacro:unless value="$(arg is_ignition)">
       <plugin filename="gz_ros2_control-system" name="gz_ros2_control::GazeboSimROS2ControlPlugin">
-        <parameters>$(find bot_controller)/config/bot_controllers.yaml</parameters>
+        <parameters>$(find bot_controller)/config/bot_controller.yaml</parameters>
       </plugin>
       <plugin filename="gz-sim-imu-system" name="gz::sim::systems::Imu">
@@ -58,5 +57,5 @@
   </gazebo>
   <!-- IMU -->
-  <!-- <gazebo reference="imu_link">
+  <gazebo reference="imu_link">
     <sensor name="imu" type="imu">
         <always_on>true</always_on>
@@ -107,4 +106,4 @@
         </imu>
     </sensor>
-  </gazebo> -->
+  </gazebo>
 </robot>

File: bot_discription/urdf/bumperbot_ros2_control.xacro (robot description, xacro)
@@ -1,4 +1,4 @@
 <?xml version="1.0"?>
-<robot xmlns:xacro="http://www.ros.org/wiki/xacro" name="bot">
+<robot xmlns:xacro="http://www.ros.org/wiki/xacro" name="bumperbot">
     <ros2_control name="RobotSystem" type="system">
         <!-- ros2_control Gazebo -->
